Commit message: Save UR10e eye-to-hand safety baseline before Foxy port

File: src/end_effector_description/urdf/end_effector_withDriverSupport.xacro (robot description, xacro)
@@ -39,10 +39,5 @@
     <origin xyz="0 -0.02 0.11" rpy="0 0 0"/>  <!-- 1cm offset from tool0 -->
   </joint>
-  <link name="camera_link"> </link>
-  <joint name="camera_joint" type="fixed">
-      <parent link="flange"/>
-      <child link="camera_link"/>
-      <!-- <origin xyz="0.0345 0 -0.1032" rpy="${pi} ${pi} ${pi}"/> -->
-      <origin xyz="0.0199931 -0.0028582 -0.109958" rpy="3.12825 -3.12574 -3.13495" />
-  </joint>
+  <!-- The calibrated camera is fixed outside the arm (eye-to-hand),
+       so it must not be attached to the moving flange. -->
 </robot>

Commit message: Make latest laboratory Foxy deployment the single main version

File: src/end_effector_description/urdf/end_effector_withDriverSupport.xacro (robot description, xacro)
@@ -1,10 +1,10 @@
 <?xml version="1.0" ?>
-<!-- displays the end-effector with UR5e(no Moveit support)-->
-<robot name="end_effector_withDriverSupport" xmlns:xacro="http://ros.org/wiki/xacro">
+<!-- UR10e and fixed end-effector for Foxy UR driver and MoveIt -->
+<robot name="$(arg name)" xmlns:xacro="http://ros.org/wiki/xacro">
   <!-- Including the claw.urdf.xacro file to give scope to xacro:claw. Inclusion is a simple copy-and-paste of code. -->
   <xacro:include filename="$(find end_effector_description)/urdf/end_effector.urdf.xacro" />
-  <!-- UR5e robot arm -->
+  <!-- UR10e robot arm -->
   <!-- URDF won't build if following args aren't defined. -->
-  <xacro:arg name="name" default="ur10e"/>
+  <xacro:arg name="name" default="ur"/>
   <xacro:arg name="ur_type" default="ur10e"/>
   <xacro:include filename="$(find ur_description)/urdf/ur.urdf.xacro"/>
@@ -39,13 +39,5 @@
     <origin xyz="0 -0.02 0.11" rpy="0 0 0"/>  <!-- 1cm offset from tool0 -->
   </joint>
-  <xacro:arg name="camera_mount" default="external"/>
-  <xacro:if value="${'$(arg camera_mount)' == 'wrist'}">
-  <link name="camera_link"> </link>
-  <joint name="camera_joint" type="fixed">
-      <parent link="flange"/>
-      <child link="camera_link"/>
-      <!-- <origin xyz="0.0345 0 -0.1032" rpy="${pi} ${pi} ${pi}"/> -->
-      <origin xyz="0.0199931 -0.0028582 -0.109958" rpy="3.12825 -3.12574 -3.13495" />
-  </joint>
-  </xacro:if>
+  <!-- The calibrated camera is fixed outside the arm (eye-to-hand),
+       so it must not be attached to the moving flange. -->
 </robot>
